File: Amp.kicad_pcb (KiCad board)
At the start: 2 copper layers, 30 x 16.8 mm, 22 parts, among them J1 MultiAV, J2 CS, J3 R, J4 G, J5 B, J6 GND, J7 +5V, U1 THS7374

Commit message: fixed some bugs
Parts:
- C2: value 100nF -> 100n; moved to F.Cu
- C3: value 22uF -> 22u; moved to F.Cu
- R10, R8: value 75 -> 38
- R9: value 75 -> 38; moved to B.Cu
- moved J8 13.9 mm to (135.1, 108.5), turned to 270 degrees
- moved C2 8.38 mm to (151.6, 109.5), turned to 90 degrees
- moved R7 3.56 mm to (142.7, 109.4)
- moved R2 2.79 mm to (144.8, 98.5)
- moved J6 2.79 mm to (126.2, 103.6)
- moved J7 2.79 mm to (126.2, 106.4)
- moved R1 2.54 mm to (147.3, 98.5), turned to 270 degrees
- moved U1 2.29 mm to (146.6, 109.6)
- moved R10 2.03 mm to (147.1, 109.4)
- moved R8 2.03 mm to (149.4, 109.4)
- moved C3 0.38 mm to (141.2, 109.2), turned to 90 degrees
- renumbered LP to J8
Connections:
- R1 pad 2: Net-(J2-Pad1) -> Net-(R1-Pad2)
- R2 pad 1: Net-(R2-Pad1) -> Net-(R1-Pad2)
- U1 pad 4: Net-(R2-Pad1) -> Net-(R1-Pad2)
Routing:
- net GND: track 90.3 -> 48.7 mm, vias 16 -> 13
- net Net-(R2-Pad1): track 17.1 -> 0.00 mm, vias 3 -> 0
- net Net-(R1-Pad2): track 0.00 -> 16.5 mm, vias 0 -> 1
- net +5V: track 33.9 -> 41.6 mm
- net Net-(J8-Pad1): track 8.99 -> 15.9 mm, vias 1 -> 2
- net Net-(R8-Pad2): track 11.1 -> 5.94 mm
- net Net-(R10-Pad2): track 8.26 -> 3.56 mm
- net Net-(J4-Pad1): track 17.4 -> 20.2 mm
- net Net-(J5-Pad1): track 15.8 -> 18.5 mm
- net Net-(J2-Pad1): track 25.7 -> 23.2 mm
- net Net-(R9-Pad2): track 6.10 -> 3.98 mm, vias 0 -> 1
- net CVIDEO_OUT: track 15.3 -> 17.1 mm
- net B_OUT: track 5.86 -> 6.49 mm
- net Net-(J3-Pad1): track 19.4 -> 19.9 mm
Other:
- board text added: "+"
- board text added: "-"
