File: Amp.sch (KiCad schematic (older format))
At the start: 22 parts, among them J1 MultiAV, J2 CS, J3 R, J4 G, J5 B, J6 GND, J7 +5V, J8 GS2, U1 THS7374

Commit message: fixed some bugs
Parts:
- R10, R8, R9: value 75 -> 38
Connections:
- net at R2.1, U1.4 (CH4_IN): now also R1.2
- net at J2.1 (Pin_1), R2.2: no longer R1.2
Other:
- moved on the sheet: J2, R2
Changed lines of the file:
@@
 P 6350 1450
 F 0 "R8" V 6430 1450 50  0000 C CNN
-F 1 "75" V 6350 1450 50  0000 C CNN
+F 1 "38" V 6350 1450 50  0000 C CNN
 F 2 "Resistors_SMD:R_1206" V 6280 1450 50  0001 C CNN
 F 3 "" H 6350 1450 50  0001 C CNN
@@
 P 6350 1600
 F 0 "R9" V 6430 1600 50  0000 C CNN
-F 1 "75" V 6350 1600 50  0000 C CNN
+F 1 "38" V 6350 1600 50  0000 C CNN
 F 2 "Resistors_SMD:R_1206" V 6280 1600 50  0001 C CNN
 F 3 "" H 6350 1600 50  0001 C CNN
@@
 P 6350 1750
 F 0 "R10" V 6430 1750 50  0000 C CNN
-F 1 "75" V 6350 1750 50  0000 C CNN
+F 1 "38" V 6350 1750 50  0000 C CNN
 F 2 "Resistors_SMD:R_1206" V 6280 1750 50  0001 C CNN
 F 3 "" H 6350 1750 50  0001 C CNN
@@
 L R R2
 U 1 1 5A20F2BA
-P 4150 1950
-F 0 "R2" V 4230 1950 50  0000 C CNN
-F 1 "4k7" V 4150 1950 50  0000 C CNN
-F 2 "Resistors_SMD:R_1206" V 4080 1950 50  0001 C CNN
-F 3 "" H 4150 1950 50  0001 C CNN
-	1    4150 1950
+P 3550 1950
+F 0 "R2" V 3630 1950 50  0000 C CNN
+F 1 "4k7" V 3550 1950 50  0000 C CNN
+F 2 "Resistors_SMD:R_1206" V 3480 1950 50  0001 C CNN
+F 3 "" H 3550 1950 50  0001 C CNN
+	1    3550 1950
 	0    1    1    0
 $EndComp
@@
 L Conn_01x01 J2
 U 1 1 5A214CB7
-P 3400 1950
-F 0 "J2" H 3400 2050 50  0000 C CNN
-F 1 "CS" H 3400 1850 50  0000 C CNN
-F 2 ".pretty:SMD_PAD_2x4" H 3400 1950 50  0001 C CNN
-F 3 "" H 3400 1950 50  0001 C CNN
-	1    3400 1950
+P 3100 1950
+F 0 "J2" H 3100 2050 50  0000 C CNN
+F 1 "CS" H 3100 1850 50  0000 C CNN
+F 2 ".pretty:SMD_PAD_2x4" H 3100 1950 50  0001 C CNN
+F 3 "" H 3100 1950 50  0001 C CNN
+	1    3100 1950
 	-1   0    0    1
 $EndComp
@@
 Wire Wire Line
 	3950 2000 3950 1950
-Wire Wire Line
-	3600 1950 4000 1950
 Connection ~ 3950 1950
 Wire Wire Line
-	4300 1950 4650 1950
+	3700 1950 4650 1950
 Wire Wire Line
 	4300 2300 3950 2300
@@
 Wire Wire Line
 	6350 2900 6400 2900
+Wire Wire Line
+	3300 1950 3400 1950
 $EndSCHEMATC
